Commit message: add interface branch files to my main branch

File: mycobot_description/urdf/mycobot/mycobot_with_d435i.urdf.xacro (robot description, xacro)
@@ -1,5 +1,10 @@
 <?xml version="1.0"?>
 <robot  xmlns:xacro="http://www.ros.org/wiki/xacro" name="mycobot" >
+  <xacro:arg name="use_nominal_extrinsics" default="false"/>
   <xacro:include filename="$(find mycobot_description)/urdf/common.xacro" />
+  <xacro:include filename="$(find realsense2_description)/urdf/_d435i.urdf.xacro" />
+  <xacro:sensor_d435i parent="link1" name="camera" use_nominal_extrinsics="$(arg use_nominal_extrinsics)">
+    <origin xyz="0.465 -0.01 0.265" rpy="0 ${pi/4} -${pi}"/>
+  </xacro:sensor_d435i>
   <link name="link1">
     <inertial>
