Commit message: change srdf and use joystick

File: mycobot_description/urdf/mycobot/mycobot_urdf.urdf (robot description, URDF)
Before this commit: robot mycobot, 7 links, 6 joints
Links:
- added link end_effector
Joints:
- added joint end_effector: type fixed, parent joint6_flange, child end_effector, origin xyz=0 0 0 rpy=0 0 0, axis 0 0 1, limit lower=-3.14 upper=3.14159 effort=1000.0 velocity=0

Commit message: add joystick control euslisp

File: mycobot_description/urdf/mycobot/mycobot_urdf.urdf (robot description, URDF)
Before this commit: robot mycobot, 8 links, 7 joints
Links:
- removed link joint1
- removed link joint2
- removed link joint3
- removed link joint4
- removed link joint5
- removed link joint6
- removed link joint6_flange
- added link link1; collision mesh filename=package://mycobot_description/urdf/mycobot/joint1.dae; visual mesh filename=package://mycobot_description/urdf/mycobot/joint1.dae
- added link link2; collision mesh filename=package://mycobot_description/urdf/mycobot/joint2.dae; visual mesh filename=package://mycobot_description/urdf/mycobot/joint2.dae
- added link link3; collision mesh filename=package://mycobot_description/urdf/mycobot/joint3.dae; visual mesh filename=package://mycobot_description/urdf/mycobot/joint3.dae
- added link link4; collision mesh filename=package://mycobot_description/urdf/mycobot/joint4.dae; visual mesh filename=package://mycobot_description/urdf/mycobot/joint4.dae
- added link link5; collision mesh filename=package://mycobot_description/urdf/mycobot/joint5.dae; visual mesh filename=package://mycobot_description/urdf/mycobot/joint5.dae
- added link link6; collision mesh filename=package://mycobot_description/urdf/mycobot/joint6.dae; visual mesh filename=package://mycobot_description/urdf/mycobot/joint6.dae
- added link link7; collision mesh filename=package://mycobot_description/urdf/mycobot/joint7.dae; visual mesh filename=package://mycobot_description/urdf/mycobot/joint7.dae
Joints:
- removed joint joint2_to_joint1
- removed joint joint3_to_joint2
- removed joint joint4_to_joint3
- removed joint joint5_to_joint4
- removed joint joint6_to_joint5
- removed joint joint6output_to_joint6
- added joint joint1: type revolute, parent link1, child link2, origin xyz=0 0 0.13156 rpy=0 0 0, axis 0 0 1, limit lower=-3.14 upper=3.14159 effort=1000.0 velocity=0
- added joint joint2: type revolute, parent link2, child link3, origin xyz=0 0  0 rpy=0 1.5708 -1.5708, axis 0 0 1, limit lower=-3.14 upper=3.14159 effort=1000.0 velocity=0
- added joint joint3: type revolute, parent link3, child link4, origin xyz=  -0.1104 0 0    rpy=0 0 0, axis  0 0 1, limit lower=-3.14 upper=3.14159 effort=1000.0 velocity=0
- added joint joint4: type revolute, parent link4, child link5, origin xyz=-0.096 0 0.06462 rpy=0 0 -1.5708, axis  0 0 1, limit lower=-3.14 upper=3.14159 effort=1000.0 velocity=0
- added joint joint5: type revolute, parent link5, child link6, origin xyz=0 -0.07318 0 rpy=1.5708 -1.5708 0, axis 0 0 1, limit lower=-3.14 upper=3.14159 effort=1000.0 velocity=0
- added joint joint6: type revolute, parent link6, child link7, origin xyz=0 0.0456 0 rpy=-1.5708 0 0, axis 0 0 1, limit lower=-3.14 upper=3.14159 effort=1000.0 velocity=0
- joint end_effector: parent joint6_flange -> link7
