Commit message: stash

File: mycobot_description/urdf/mycobot/mycobot_with_gripper_parallel.urdf (robot description, URDF)
Before this commit: robot mycobot, 15 links, 14 joints
Joints:
- removed joint g_base_to_joint1
- removed joint joint6output_to_gripper_base
- added joint g_base_to_link1: type fixed, parent g_base, child link1, origin xyz=0 0 0 rpy=0 0 0, axis 0 0 0, limit lower=-3.14 upper=3.14159 effort=1000.0 velocity=0
- added joint link7_to_gripper_base: type fixed, parent link7, child gripper_base, origin xyz=0 0 0.034 rpy=1.579 0 0

Commit message: update

File: mycobot_description/urdf/mycobot/mycobot_with_gripper_parallel.urdf (robot description, URDF)
Before this commit: robot mycobot, 15 links, 14 joints
Joints:
- joint link7_to_gripper_base: origin xyz=0 0 0.034 rpy=1.579 0 0 -> xyz=0 0 0.034 rpy=${pi/2} 0 ${-pi/4}

Commit message: Revert "update"
This reverts commit 7c478ecd22c5dd44293ac05b854715755e38dd6b.

File: mycobot_description/urdf/mycobot/mycobot_with_gripper_parallel.urdf (robot description, URDF)
Before this commit: robot mycobot, 15 links, 14 joints
Joints:
- joint link7_to_gripper_base: origin xyz=0 0 0.034 rpy=${pi/2} 0 ${-pi/4} -> xyz=0 0 0.034 rpy=1.579 0 0
