Commit message: mycobot-mujoco-project

File: mycobot_description/urdf/mycobot/mycobot.urdf (robot description, URDF)
Before this commit: robot mycobot, 8 links, 7 joints
Links:
- link link1: geometry collision mesh filename=package://mycobot_description/urdf/mycobot/mesh/link1.obj; visual mesh filename=package://mycobot_description/urdf/mycobot/mesh/link1.obj
- link link2: geometry collision mesh filename=package://mycobot_description/urdf/mycobot/mesh/link2.obj; visual mesh filename=package://mycobot_description/urdf/mycobot/mesh/link2.obj
- link link3: geometry collision mesh filename=package://mycobot_description/urdf/mycobot/mesh/link3.obj; visual mesh filename=package://mycobot_description/urdf/mycobot/mesh/link3.obj
- link link4: geometry collision mesh filename=package://mycobot_description/urdf/mycobot/mesh/link4.obj; visual mesh filename=package://mycobot_description/urdf/mycobot/mesh/link4.obj
- link link5: geometry collision mesh filename=package://mycobot_description/urdf/mycobot/mesh/link5.obj; visual mesh filename=package://mycobot_description/urdf/mycobot/mesh/link5.obj
- link link6: geometry collision mesh filename=package://mycobot_description/urdf/mycobot/mesh/link6.obj; visual mesh filename=package://mycobot_description/urdf/mycobot/mesh/link6.obj
- link link7: geometry collision mesh filename=package://mycobot_description/urdf/mycobot/mesh/link7.obj; visual mesh filename=package://mycobot_description/urdf/mycobot/mesh/link7.obj
