Commit message: for dual arm

File: mycobot_description/urdf/mycobot/mycobot_with_gripper_dae.urdf.xacro (robot description, xacro)
@@ -195,5 +195,5 @@
       <geometry>
        <!--- 0.0 0 -0.04 -->
-       <mesh filename="package://mycobot_description/urdf/mycobot/mesh/gripper_base.obj"/>
+       <mesh filename="package://mycobot_description/urdf/mycobot/mesh/gripper_base.dae"/>
       </geometry>
     <origin xyz = "0.0 0.008 -0.012 " rpy = " 0 0 0"/>
@@ -202,5 +202,5 @@
       <geometry>
        <!--- 0.0 0 -0.04 -->
-       <mesh filename="package://mycobot_description/urdf/mycobot/mesh/gripper_base.obj"/>
+       <mesh filename="package://mycobot_description/urdf/mycobot/mesh/gripper_base.dae"/>
       </geometry>
     <origin xyz = "0.0 0.008 -0.012 " rpy = " 0 0 0"/>
@@ -211,5 +211,5 @@
       <geometry>
        <!--- 0.0 0 -0.04 -->
-       <mesh filename="package://mycobot_description/urdf/mycobot/mesh/gripper_left1.obj"/>
+       <mesh filename="package://mycobot_description/urdf/mycobot/mesh/gripper_left1.dae"/>
       </geometry>
     <origin xyz = "0.039 -0.0133 -0.012 " rpy = " 0 0 0"/>
@@ -218,5 +218,5 @@
     <collision>
       <geometry>
-       <mesh filename="package://mycobot_description/urdf/mycobot/mesh/gripper_left1.obj"/>
+       <mesh filename="package://mycobot_description/urdf/mycobot/mesh/gripper_left1.dae"/>
       </geometry>
         <origin xyz = "0.039 -0.0133 -0.012 " rpy = " 0 0 0"/>
@@ -226,5 +226,5 @@
     <visual>
       <geometry>
-       <mesh filename="package://mycobot_description/urdf/mycobot/mesh/gripper_left2.obj"/>
+       <mesh filename="package://mycobot_description/urdf/mycobot/mesh/gripper_left2.dae"/>
       </geometry>
     <origin xyz = "0.005 -0.0195 -0.012 " rpy = " 0 0 0"/>
@@ -232,5 +232,5 @@
     <collision>
       <geometry>
-       <mesh filename="package://mycobot_description/urdf/mycobot/mesh/gripper_left2.obj"/>
+       <mesh filename="package://mycobot_description/urdf/mycobot/mesh/gripper_left2.dae"/>
       </geometry>
         <origin xyz = "0.005 -0.0195 -0.012 " rpy = " 0 0 0"/>
@@ -240,5 +240,5 @@
     <visual>
       <geometry>
-       <mesh filename="package://mycobot_description/urdf/mycobot/mesh/gripper_left3.obj"/>
+       <mesh filename="package://mycobot_description/urdf/mycobot/mesh/gripper_left3.dae"/>
       </geometry>
     <origin xyz = "0.012 0.0025 -0.012 " rpy = " 0 0 0"/>
@@ -247,5 +247,5 @@
     <collision>
       <geometry>
-       <mesh filename="package://mycobot_description/urdf/mycobot/mesh/gripper_left3.obj"/>
+       <mesh filename="package://mycobot_description/urdf/mycobot/mesh/gripper_left3.dae"/>
       </geometry>
     <origin xyz = "0.0 0 -0.012 " rpy = " 0 0 0"/>
@@ -255,5 +255,5 @@
     <visual>
       <geometry>
-       <mesh filename="package://mycobot_description/urdf/mycobot/mesh/gripper_right1.obj"/>
+       <mesh filename="package://mycobot_description/urdf/mycobot/mesh/gripper_right1.dae"/>
       </geometry>
     <origin xyz = "-0.039 -0.0133 -0.012 " rpy = " 0 0 0"/>
@@ -261,5 +261,5 @@
     <collision>
       <geometry>
-       <mesh filename="package://mycobot_description/urdf/mycobot/mesh/gripper_right1.obj"/>
+       <mesh filename="package://mycobot_description/urdf/mycobot/mesh/gripper_right1.dae"/>
       </geometry>
         <origin xyz = "-0.039 -0.0133 -0.012 " rpy = " 0 0 0"/>
@@ -269,5 +269,5 @@
     <visual>
       <geometry>
-       <mesh filename="package://mycobot_description/urdf/mycobot/mesh/gripper_right2.obj"/>
+       <mesh filename="package://mycobot_description/urdf/mycobot/mesh/gripper_right2.dae"/>
       </geometry>
     <origin xyz = "-0.005 -0.0195 -0.012 " rpy = " 0 0 0"/>
@@ -275,5 +275,5 @@
     <collision>
       <geometry>
-       <mesh filename="package://mycobot_description/urdf/mycobot/mesh/gripper_right2.obj"/>
+       <mesh filename="package://mycobot_description/urdf/mycobot/mesh/gripper_right2.dae"/>
       </geometry>
         <origin xyz = "-0.005 -0.0195 -0.012 " rpy = " 0 0 0"/>
@@ -283,5 +283,5 @@
     <visual>
       <geometry>
-       <mesh filename="package://mycobot_description/urdf/mycobot/mesh/gripper_right3.obj"/>
+       <mesh filename="package://mycobot_description/urdf/mycobot/mesh/gripper_right3.dae"/>
       </geometry>
     <origin xyz = "-0.012 0.0025 -0.012 " rpy = " 0 0 0"/>
@@ -289,5 +289,5 @@
     <collision>
       <geometry>
-       <mesh filename="package://mycobot_description/urdf/mycobot/mesh/gripper_right3.obj"/>
+       <mesh filename="package://mycobot_description/urdf/mycobot/mesh/gripper_right3.dae"/>
       </geometry>
     <origin xyz = "-0.012 0.0025 -0.012" rpy = " 0 0 0"/>
