Commit message: add gripper on mujoco

File: mycobot_description/urdf/mycobot/mycobot.urdf.xacro (robot description, xacro)
@@ -143,10 +143,4 @@
     </collision>
   </link>
-  <link name="camera_link"/>
-  <joint name="camera" type="fixed">
-      <parent link="link1"/>
-      <child link="camera_link"/>
-      <origin xyz = "0.36 0 0.57 " rpy = "0 0 0"/>
-  </joint>
   <joint name="joint1" type="revolute">
     <axis xyz="0 0 1"/>

Commit message: changed correct limit joints

File: mycobot_description/urdf/mycobot/mycobot.urdf.xacro (robot description, xacro)
@@ -145,5 +145,5 @@
   <joint name="joint1" type="revolute">
     <axis xyz="0 0 1"/>
-    <limit effort = "10.0" lower = "${-pi}" upper = "${pi}" velocity = "1.0"/>
+    <limit effort = "10.0" lower = "${-pi/180*165}" upper = "${pi/180*165}" velocity = "1.0"/>
     <parent link="link1"/>
     <child link="link2"/>
@@ -153,5 +153,5 @@
   <joint name="joint2" type="revolute">
     <axis xyz="0 0 1"/>
-    <limit effort = "10.0" lower = "${-pi}" upper = "${pi}" velocity = "1.0"/>
+    <limit effort = "10.0" lower = "${-pi/180*165}" upper = "${pi/180*165}" velocity = "1.0"/>
     <parent link="link2"/>
     <child link="link3"/>
@@ -161,5 +161,5 @@
   <joint name="joint3" type="revolute">
     <axis xyz=" 0 0 1"/>
-    <limit effort = "10.0" lower = "${-pi}" upper = "${pi}" velocity = "1.0"/>
+    <limit effort = "10.0" lower = "${-pi/180*165}" upper = "${pi/180*165}" velocity = "1.0"/>
     <parent link="link3"/>
     <child link="link4"/>
@@ -169,5 +169,5 @@
   <joint name="joint4" type="revolute">
     <axis xyz=" 0 0 1"/>
-    <limit effort = "10.0" lower = "${-pi}" upper = "${pi}" velocity = "1.0"/>
+    <limit effort = "10.0" lower = "${-pi/180*165}" upper = "${pi/180*165}" velocity = "1.0"/>
     <parent link="link4"/>
     <child link="link5"/>
@@ -177,5 +177,5 @@
   <joint name="joint5" type="revolute">
     <axis xyz="0 0 1"/>
-    <limit effort = "10.0" lower = "${-pi}" upper = "${pi}" velocity = "1.0"/>
+    <limit effort = "10.0" lower = "${-pi/180*165}" upper = "${pi/180*165}" velocity = "1.0"/>
     <parent link="link5"/>
     <child link="link6"/>
@@ -185,5 +185,5 @@
   <joint name="joint6" type="revolute">
     <axis xyz="0 0 1"/>
-    <limit effort = "10.0" lower = "${-pi}" upper = "${pi}" velocity = "1.0"/>
+    <limit effort = "10.0" lower = "${-pi/180*175}" upper = "${pi/180*175}" velocity = "1.0"/>
     <parent link="link6"/>
     <child link="link7"/>
